Commit message: feat(motion): implement Phase 3B differential-drive motion and /cmd_vel bridge in Gazebo Fortress

File: src/ugv_navigation/urdf/ugv.urdf.xacro (robot description, xacro)
@@ -12,4 +12,5 @@
   <xacro:property name="wheel_y_offset" value="0.25" />
   <xacro:property name="wheel_z_offset" value="-0.05" />
+  <xacro:property name="track_width" value="${wheel_y_offset * 2.0}" />
   <xacro:property name="base_link_z_offset" value="0.15" />
   <!-- Inertia Helper Macros -->
@@ -172,3 +173,27 @@
     <origin xyz="0.0 0.0 0.0" rpy="0 0 0" />
   </joint>
+  <!-- Gazebo Fortress Differential / Skid-Steer Drive Plugin -->
+  <gazebo>
+    <plugin filename="ignition-gazebo-diff-drive-system" name="gz::sim::systems::DiffDrive">
+      <!-- Wheel Joints -->
+      <left_joint>front_left_wheel_joint</left_joint>
+      <left_joint>rear_left_wheel_joint</left_joint>
+      <right_joint>front_right_wheel_joint</right_joint>
+      <right_joint>rear_right_wheel_joint</right_joint>
+      <!-- Kinematic Parameters -->
+      <wheel_separation>${track_width}</wheel_separation>
+      <wheel_radius>${wheel_radius}</wheel_radius>
+      <!-- Dynamic Limits -->
+      <max_linear_acceleration>2.5</max_linear_acceleration>
+      <min_linear_acceleration>-2.5</min_linear_acceleration>
+      <max_angular_acceleration>3.0</max_angular_acceleration>
+      <min_angular_acceleration>-3.0</min_angular_acceleration>
+      <max_linear_velocity>1.5</max_linear_velocity>
+      <min_linear_velocity>-1.5</min_linear_velocity>
+      <max_angular_velocity>2.0</max_angular_velocity>
+      <min_angular_velocity>-2.0</min_angular_velocity>
+      <!-- Motion Command Topic -->
+      <topic>/cmd_vel</topic>
+    </plugin>
+  </gazebo>
 </robot>

Commit message: feat(sensors): implement Phase 3D camera/LiDAR/IMU sensors with ogre2 rendering and bridge them to ROS 2

File: src/ugv_navigation/urdf/ugv.urdf.xacro (robot description, xacro)
@@ -121,10 +121,4 @@
       <material name="camera_mat" />
     </visual>
-    <collision>
-      <origin xyz="0 0 0" rpy="0 0 0" />
-      <geometry>
-        <box size="0.04 0.06 0.03" />
-      </geometry>
-    </collision>
   </link>
   <joint name="camera_joint" type="fixed">
@@ -135,4 +129,22 @@
   <gazebo reference="camera_link">
     <material>Gazebo/Red</material>
+    <sensor name="camera_sensor" type="camera">
+      <always_on>1</always_on>
+      <update_rate>20</update_rate>
+      <visualize>false</visualize>
+      <topic>camera</topic>
+      <camera name="camera">
+        <optical_frame_id>camera_optical_frame</optical_frame_id>
+        <horizontal_fov>1.3962634</horizontal_fov>
+        <image>
+          <width>640</width>
+          <height>480</height>
+        </image>
+        <clip>
+          <near>0.1</near>
+          <far>100</far>
+        </clip>
+      </camera>
+    </sensor>
   </gazebo>
   <link name="camera_optical_frame" />
@@ -143,26 +155,40 @@
   </joint>
   <!-- LiDAR mount -->
-  <link name="lidar_link">
-    <visual>
-      <origin xyz="0 0 0" rpy="0 0 0" />
-      <geometry>
-        <cylinder radius="0.04" length="0.05" />
-      </geometry>
-      <material name="lidar_mat" />
-    </visual>
-    <collision>
-      <origin xyz="0 0 0" rpy="0 0 0" />
-      <geometry>
-        <cylinder radius="0.04" length="0.05" />
-      </geometry>
-    </collision>
-  </link>
+  <link name="lidar_link" />
   <joint name="lidar_joint" type="fixed">
     <parent link="base_link" />
     <child link="lidar_link" />
-    <origin xyz="0.0 0.0 ${chassis_height/2.0 + 0.025}" rpy="0 0 0" />
+    <origin xyz="0.0 0.0 ${chassis_height/2.0 + 0.125}" rpy="0 0 0" />
   </joint>
   <gazebo reference="lidar_link">
     <material>Gazebo/Black</material>
+    <sensor name="gpu_lidar_sensor" type="gpu_lidar">
+      <always_on>1</always_on>
+      <update_rate>20</update_rate>
+      <visualize>false</visualize>
+      <topic>scan</topic>
+      <ignition_frame_id>lidar_link</ignition_frame_id>
+      <lidar>
+        <scan>
+          <horizontal>
+            <samples>360</samples>
+            <resolution>1</resolution>
+            <min_angle>-3.14159265358979</min_angle>
+            <max_angle>3.14159265358979</max_angle>
+          </horizontal>
+          <vertical>
+            <samples>1</samples>
+            <resolution>1</resolution>
+            <min_angle>0.0</min_angle>
+            <max_angle>0.0</max_angle>
+          </vertical>
+        </scan>
+        <range>
+          <min>0.1</min>
+          <max>20.0</max>
+          <resolution>0.01</resolution>
+        </range>
+      </lidar>
+    </sensor>
   </gazebo>
   <!-- IMU link -->
@@ -173,4 +199,13 @@
     <origin xyz="0.0 0.0 0.0" rpy="0 0 0" />
   </joint>
+  <gazebo reference="imu_link">
+    <sensor name="imu_sensor" type="imu">
+      <always_on>1</always_on>
+      <update_rate>100</update_rate>
+      <visualize>false</visualize>
+      <topic>imu</topic>
+      <ignition_frame_id>imu_link</ignition_frame_id>
+    </sensor>
+  </gazebo>
   <!-- Gazebo Fortress Differential / Skid-Steer Drive Plugin -->
   <gazebo>
